File: 2020/AtmelPcb/eagle/hviezda.brd (EAGLE design)
At the start: 94.3 x 90.2 mm, 15 parts, among them U1 ATTINY84-20PU

Commit message: blikajuca hviezda update
Parts:
- moved BAT1 19.3 mm to (10.2, 41.9)
- moved C1 19.3 mm to (26.7, 50.8)
- moved LED1 19.3 mm to (45.7, 10.2)
- moved LED2 19.3 mm to (6.99, 10.2)
- moved LED3 19.3 mm to (57.8, 47.0)
- moved LED4 19.3 mm to (26.7, 69.8)
- moved LED5 19.3 mm to (-5.08, 47.0)
- moved R1 19.3 mm to (40.6, 35.6)
- moved R2 19.3 mm to (40.6, 39.4)
- moved R3 19.3 mm to (40.6, 43.2)
- moved R4 19.3 mm to (40.6, 47.0)
- moved R5 19.3 mm to (11.4, 17.8)
- moved S1 19.3 mm to (26.7, 58.4)
- moved SV1 19.3 mm to (26.7, 24.1)
- moved U1 19.3 mm to (30.5, 31.8)
Routing:
- net N$10: track 25.0 -> 26.8 mm
Other:
- outline, holes or cut-outs redrawn
