File: 2020/AtmelPcb/eagle/hviezda.sch (EAGLE design)
At the start: 15 parts, among them U1 ATTINY84-20PU

Commit message: blikajuca hviezda update
Other:
- moved on the sheet: BAT1
Changed lines of the file:
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@@
 <attribute name="VALUE" x="25.019" y="11.684" size="1.778" layer="96" rot="R90"/>
 </instance>
-<instance part="BAT1" gate="1" x="40.64" y="15.24" smashed="yes">
-<attribute name="NAME" x="35.56" y="20.32" size="1.778" layer="95" rot="MR180"/>
-<attribute name="VALUE" x="35.56" y="10.16" size="1.778" layer="95"/>
+<instance part="BAT1" gate="1" x="22.86" y="20.32" smashed="yes">
+<attribute name="NAME" x="17.78" y="25.4" size="1.778" layer="95" rot="MR180"/>
+<attribute name="VALUE" x="17.78" y="15.24" size="1.778" layer="95"/>
 </instance>
 </instances>
@@
 </segment>
 <segment>
-<wire x1="45.72" y1="15.24" x2="55.88" y2="15.24" width="0.1524" layer="91"/>
+<wire x1="27.94" y1="20.32" x2="30.48" y2="20.32" width="0.1524" layer="91"/>
 <pinref part="BAT1" gate="1" pin="+"/>
 </segment>
@@
 </segment>
 <segment>
-<wire x1="17.78" y1="10.16" x2="10.16" y2="10.16" width="0.1524" layer="91"/>
+<wire x1="17.78" y1="10.16" x2="12.7" y2="10.16" width="0.1524" layer="91"/>
 <pinref part="C1" gate="G$1" pin="1"/>
 </segment>
 <segment>
-<wire x1="35.56" y1="15.24" x2="27.94" y2="15.24" width="0.1524" layer="91"/>
+<wire x1="17.78" y1="20.32" x2="15.24" y2="20.32" width="0.1524" layer="91"/>
 <pinref part="BAT1" gate="1" pin="-"/>
 </segment>
@@
 <pinref part="U1" gate="A" pin="PB0"/>
 <wire x1="-25.4" y1="58.42" x2="-45.72" y2="58.42" width="0.1524" layer="91"/>
-<wire x1="-45.72" y1="58.42" x2="-45.72" y2="35.56" width="0.1524" layer="91"/>
-<wire x1="-45.72" y1="35.56" x2="22.86" y2="35.56" width="0.1524" layer="91"/>
+<wire x1="-45.72" y1="58.42" x2="-45.72" y2="33.02" width="0.1524" layer="91"/>
+<wire x1="-45.72" y1="33.02" x2="27.94" y2="33.02" width="0.1524" layer="91"/>
 <pinref part="S1" gate="1" pin="P1"/>
-<wire x1="27.94" y1="33.02" x2="22.86" y2="33.02" width="0.1524" layer="91"/>
-<wire x1="22.86" y1="33.02" x2="22.86" y2="35.56" width="0.1524" layer="91"/>
-</segment>
-</net>
+</segment>
+</net>
